Commit message: spawn model using gazebo service

File: swarm_robot_description/urdf/enclosure_side_customization.urdf (robot description, URDF)
Before this commit: robot unit_enclosure, 5 links, 4 joints
Links:
- removed link x+1
- removed link x-1
- removed link y+1
- removed link y-1
- added link x_lower, mass 1; collision box size=0.05 2.1 0.05; visual box size=0.05 2.1 0.05
- added link x_upper, mass 1; collision box size=0.05 2.1 0.05; visual box size=0.05 2.1 0.05
- added link y_lower, mass 1; collision box size=2.0 0.05 0.05; visual box size=2.0 0.05 0.05
- added link y_upper, mass 1; collision box size=2.0 0.05 0.05; visual box size=2.0 0.05 0.05
Joints:
- removed joint glue_wall_x+1
- removed joint glue_wall_x-1
- removed joint glue_wall_y+1
- removed joint glue_wall_y-1
- added joint glue_wall_x_lower: type fixed, parent world, child x_lower, origin xyz=-1.025 0 0.025 rpy=0 0 0
- added joint glue_wall_x_upper: type fixed, parent world, child x_upper, origin xyz=1.025 0 0.025 rpy=0 0 0
- added joint glue_wall_y_lower: type fixed, parent world, child y_lower, origin xyz=0 -1.025 0.025 rpy=0 0 0
- added joint glue_wall_y_upper: type fixed, parent world, child y_upper, origin xyz=0 1.025 0.025 rpy=0 0 0
