Commit message: successfully spawn multiple robots in gazebo randomly

File: swarm_robot_description/urdf/enclosure_halfside_3.0.urdf (robot description, URDF)
Before this commit: robot enclosure_side_customization, 5 links, 4 joints
Links:
- link x_lower: geometry collision box size=0.05 6.1 0.05; visual box size=0.05 6.1 0.05
- link x_upper: geometry collision box size=0.05 6.1 0.05; visual box size=0.05 6.1 0.05
- link y_lower: geometry collision box size=6.0 0.05 0.05; visual box size=6.0 0.05 0.05
- link y_upper: geometry collision box size=6.0 0.05 0.05; visual box size=6.0 0.05 0.05
Joints:
- joint glue_wall_x_lower: origin xyz=-1.025 0 0.025 rpy=0 0 0 -> xyz=-3.025 0 0.025 rpy=0 0 0
- joint glue_wall_x_upper: origin xyz=1.025 0 0.025 rpy=0 0 0 -> xyz=3.025 0 0.025 rpy=0 0 0
- joint glue_wall_y_lower: origin xyz=0 -1.025 0.025 rpy=0 0 0 -> xyz=0 -3.025 0.025 rpy=0 0 0
- joint glue_wall_y_upper: origin xyz=0 1.025 0.025 rpy=0 0 0 -> xyz=0 3.025 0.025 rpy=0 0 0
