Commit message: fix some parameters in two_wheel_robot.urdf

File: swarm_robot_description/urdf/two_wheel_robot.urdf (robot description, URDF)
Before this commit: robot two_wheel_robot, 3 links, 2 joints
Joints:
- joint left_motor: origin xyz=0 -0.0177 0.015 rpy=-1.5708 0 0 -> xyz=0 -0.0177 0.0127 rpy=-1.5708 0 0
- joint right_motor: origin xyz=0 0.0177 0.015 rpy=1.5708 0 0 -> xyz=0 0.0177 0.0127 rpy=1.5708 0 0

Commit message: increase body inertia of two wheel robot

File: swarm_robot_description/urdf/two_wheel_robot.urdf (robot description, URDF)
Before this commit: robot two_wheel_robot, 3 links, 2 joints
Links:
- link left_wheel: mass 0.001 -> 0.002; geometry collision cylinder length=0.004 radius=0.015; visual cylinder length=0.004 radius=0.015
- link right_wheel: mass 0.001 -> 0.002; geometry collision cylinder length=0.004 radius=0.015; visual cylinder length=0.004 radius=0.015

Commit message: fix urdf errors with respect to description in gazebo

File: swarm_robot_description/urdf/two_wheel_robot.urdf (robot description, URDF)
Before this commit: robot two_wheel_robot, 3 links, 2 joints
Joints:
- joint left_motor: origin xyz=0 -0.0177 0.0127 rpy=-1.5708 0 0 -> xyz=0 0.0177 0.0127 rpy=1.5708 0 0
- joint right_motor: origin xyz=0 0.0177 0.0127 rpy=1.5708 0 0 -> xyz=0 -0.0177 0.0127 rpy=-1.5708 0 0

Commit message: important change at robot model, tuned the wheel direction

File: swarm_robot_description/urdf/two_wheel_robot.urdf (robot description, URDF)
Before this commit: robot two_wheel_robot, 3 links, 2 joints
Joints:
- joint left_motor: axis 0 0 1 -> 0 0 -1

Commit message: add collada files for two wheel robot

File: swarm_robot_description/urdf/two_wheel_robot.urdf (robot description, URDF)
Before this commit: robot two_wheel_robot, 3 links, 2 joints
Links:
- link body_link: geometry collision mesh filename=package://swarm_robot_description/sketchup/twowheel_body.dae; visual mesh filename=package://swarm_robot_description/sketchup/twowheel_body.dae
- link left_wheel: geometry collision mesh filename=package://swarm_robot_description/sketchup/twowheel_left.dae; visual mesh filename=package://swarm_robot_description/sketchup/twowheel_left.dae
- link right_wheel: geometry collision mesh filename=package://swarm_robot_description/sketchup/twowheel_right.d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; visual mesh filename=package://swarm_robot_description/sketchup/twowheel_right.d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

Commit message: add sphere support for two wheel robot

File: swarm_robot_description/urdf/two_wheel_robot.urdf (robot description, URDF)
Before this commit: robot two_wheel_robot, 3 links, 2 joints
Links:
- added link back_sphere, mass 0.0000001; collision sphere radius=0.002298
- added link front_sphere, mass 0.0000001; collision sphere radius=0.002298
Joints:
- added joint back_support: type fixed, parent body_link, child back_sphere, origin xyz=-0.0104 0 0 rpy=0 0 0
- added joint front_support: type fixed, parent body_link, child front_sphere, origin xyz=0.0104 0 0 rpy=0 0 0

Commit message: update mesh file

File: swarm_robot_description/urdf/two_wheel_robot.urdf (robot description, URDF)
Before this commit: robot two_wheel_robot, 5 links, 4 joints
Links:
- link body_link: geometry collision mesh filename=package://swarm_robot_description/urdf/mesh/twowheel_body.d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; visual mesh filename=package://swarm_robot_description/urdf/mesh/twowheel_body.d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
- link left_wheel: geometry collision mesh filename=package://swarm_robot_description/urdf/mesh/twowheel_left.d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; visual mesh filename=package://swarm_robot_description/urdf/mesh/twowheel_left.d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
- link right_wheel: geometry collision mesh filename=package://swarm_robot_description/urdf/mesh/twowheel_right.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; visual mesh filename=package://swarm_robot_description/urdf/mesh/twowheel_right.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

Commit message: update two wheel robot model

File: swarm_robot_description/urdf/two_wheel_robot.urdf (robot description, URDF)
Before this commit: robot two_wheel_robot, 5 links, 4 joints
Links:
- added link left_wheel_mark, mass 0.0000001; collision mesh filename=package://swarm_robot_description/urdf/mesh/twowheel_left_m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; visual mesh filename=package://swarm_robot_description/urdf/mesh/twowheel_left_m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
- link left_wheel: geometry collision cylinder length=0.004 radius=0.015; visual cylinder length=0.004 radius=0.015
- link right_wheel: geometry collision cylinder length=0.004 radius=0.015; visual cylinder length=0.004 radius=0.015
Joints:
- added joint left_wheel_mark_fixed: type continuous, parent left_wheel, child left_wheel_mark, origin xyz=0 0 0.014 rpy=0 0 0, axis 0 0 1
- joint left_motor: origin xyz=0 0.0177 0.0127 rpy=1.5708 0 0 -> xyz=0 0.0137 0.0127 rpy=-1.5708 0 0
- joint right_motor: origin xyz=0 -0.0177 0.0127 rpy=-1.5708 0 0 -> xyz=0 -0.0137 0.0127 rpy=1.5708 0 0

Commit message: update robot model mesh files

File: swarm_robot_description/urdf/two_wheel_robot.urdf (robot description, URDF)
Before this commit: robot two_wheel_robot, 6 links, 5 joints
Links:
- removed link left_wheel_mark
- link back_sphere: geometry collision sphere radius=0.002297
- link front_sphere: geometry collision sphere radius=0.002297
- link left_wheel: geometry collision cylinder length=0.004 radius=0.015; visual mesh filename=package://swarm_robot_description/urdf/mesh/twowheel_left_l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
- link right_wheel: geometry collision cylinder length=0.004 radius=0.015; visual mesh filename=package://swarm_robot_description/urdf/mesh/twowheel_right_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
Joints:
- removed joint left_wheel_mark_fixed

Commit message: finish debugging the batch adding node

File: swarm_robot_description/urdf/two_wheel_robot.urdf (robot description, URDF)
Before this commit: robot two_wheel_robot, 5 links, 4 joints
Links:
- link left_wheel: geometry collision cylinder length=0.004 radius=0.015; visual cylinder length=0.004 radius=0.015
- link right_wheel: geometry collision cylinder length=0.004 radius=0.015; visual cylinder length=0.004 radius=0.015

Commit message: fix wheel robot rotation axis

File: swarm_robot_description/urdf/two_wheel_robot.urdf (robot description, URDF)
Before this commit: robot two_wheel_robot, 5 links, 4 joints
Links:
- link left_wheel: geometry collision cylinder length=0.004 radius=0.015; visual mesh filename=package://swarm_robot_description/urdf/mesh/twowheel_left_l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
- link right_wheel: geometry collision cylinder length=0.004 radius=0.015; visual mesh filename=package://swarm_robot_description/urdf/mesh/twowheel_right_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
Joints:
- joint left_motor: axis 0 0 -1 -> 0 0 1
- joint right_motor: axis 0 0 1 -> 0 0 -1
